File: alps-rk27.kicad_pcb (KiCad board)
At the start: 2 copper layers, 44 x 48 mm, 7 parts, among them J1 ONE, J2 TWO

Commit message: Prepare for fab
Other:
- board text added: "IN"
- board text added: "OUT"
- board text removed: "IN1"
- board text removed: "IN2"
- board text removed: "OUT1"
- board text removed: "OUT2"
Changed lines of the file:
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@@
 		)
 	)
-	(gr_text "OUT1"
+	(gr_text "OUT"
 		(at 135.2 105.9 180)
 		(layer "B.SilkS")
@@
 		)
 	)
-	(gr_text "IN2"
+	(gr_text "IN"
 		(at 135.3 87 180)
 		(layer "B.SilkS")
@@
 		)
 	)
-	(gr_text "OUT2"
+	(gr_text "OUT"
 		(at 135.3 89.6 180)
 		(layer "B.SilkS")
@@
 		)
 	)
-	(gr_text "IN1"
+	(gr_text "IN"
 		(at 135.3 103.4 180)
 		(layer "B.SilkS")
@@
 			(justify left bottom mirror)
 		)
-	)
-	(segment
-		(start 153.9 94.3)
-		(end 153.9 107.35)
-		(width 1.5)
-		(layer "F.Cu")
-		(net "IN_2")
-	)
-	(segment
-		(start 146.7 87.1)
-		(end 153.9 94.3)
-		(width 1.5)
-		(layer "F.Cu")
-		(net "IN_2")
-	)
-	(segment
-		(start 129.5 87.1)
-		(end 146.7 87.1)
-		(width 1.5)
-		(layer "F.Cu")
-		(net "IN_2")
 	)
 	(segment
@@
 		(net "OUT_2")
 	)
+	(segment
+		(start 153.9 94.3)
+		(end 153.9 107.35)
+		(width 1.5)
+		(layer "F.Cu")
+		(net "IN_2")
+	)
+	(segment
+		(start 146.7 87.1)
+		(end 153.9 94.3)
+		(width 1.5)
+		(layer "F.Cu")
+		(net "IN_2")
+	)
+	(segment
+		(start 129.5 87.1)
+		(end 146.7 87.1)
+		(width 1.5)
+		(layer "F.Cu")
+		(net "IN_2")
+	)
 	(zone
